Commit message: depth camera integration

File: description/lidar.xacro (robot description, xacro)
@@ -23,4 +23,5 @@
 </link>
 <gazebo reference="laser_frame">
+    <material>Gazebo/Red</material>
     <sensor name="laser" type="ray">
         <pose>0 0 0 0 0 0</pose>

File: description/robot.urdf.xacro (robot description, xacro)
@@ -4,3 +4,5 @@
 <xacro:include filename="gazebo_control.xacro"/>
 <xacro:include filename="lidar.xacro"/>
+<!--    <xacro:include filename="camera.xacro"/>    -->
+<xacro:include filename="depth_camera.xacro"/>
 </robot>
